Commit message: Added meshes

File: elektron_defs/robots/elektron.udrf.xacro (robot description, xacro)
@@ -20,8 +20,9 @@
                izz="1.0" />
     </inertial>
+        <!--<box size="0.38 0.28 0.20" />-->
     <visual>
       <origin xyz="-0.0 0 0.115" rpy="0 0 0" />
       <geometry>
-        <box size="0.38 0.28 0.20" />
+        <mesh filename="package://elektron_defs/meshes/elektron_body.blend"/>
       </geometry>
     </visual>

Commit message: .xacro file cleanup

File: elektron_defs/robots/elektron.udrf.xacro (robot description, xacro)
@@ -1,162 +1,162 @@
 <?xml version="1.0"?>
-<robot name="elektron"
-       xmlns:sensor="http://playerstage.sourceforge.net/gazebo/xmlschema/#sensor"
-       xmlns:controller="http://playerstage.sourceforge.net/gazebo/xmlschema/#controller"
-       xmlns:xacro="http://ros.org/wiki/fixme"
-       xmlns:interface="http://playerstage.sourceforge.net/gazebo/xmlschema/#interface">
-  <property name="M_PI" value="3.14159"/>
-  <property name="base_size_x" value="0.38" />
-  <property name="base_size_y" value="0.28" />
-  <property name="base_size_z" value="0.18" />
-  <property name="wheel_radius" value="0.05" />
-  <property name="wheel_length" value="0.02" />
-  <property name="caster_wheel_offset_y" value="0.1675" />
-  <link name="base_link">
-    <inertial>
-      <mass value="15" />
-      <origin xyz="-0.0 0 ${base_size_z/2}" />
-      <inertia ixx="1.0" ixy="0.0" ixz="0.0"
-               iyy="1.0" iyz="0.0"
-               izz="1.0" />
-    </inertial>
-        <!--<box size="0.38 0.28 0.20" />-->
-    <visual>
-      <origin xyz="-0.0 0 0.115" rpy="0 0 0" />
-      <geometry>
-        <mesh filename="package://elektron_defs/meshes/elektron_body.blend"/>
-      </geometry>
-    </visual>
-    <collision>
-      <origin xyz="-0.0 0 0.115" rpy="0 0 0" />
-      <geometry>
-        <box size="0.30 0.28 0.20" />
-      </geometry>
-      <material name="Cyan">
-        <color rgba="0 255 255 1.0"/>
-      </material>
-    </collision>
-  </link>
-  <xacro:macro name="erratic_wheel" params="suffix parent reflect offset m">
-    <joint name="${parent}_${suffix}_wheel_joint" type="continuous">
-      <origin xyz="${offset} ${reflect*caster_wheel_offset_y} ${wheel_radius}" rpy="0 0 0" />
-      <axis xyz="0 1 0" />
-      <anchor xyz="0 0 0" />
-      <limit effort="100" velocity="100" />
-      <joint_properties damping="0.0" friction="0.0" />
-      <parent link="${parent}" />
-      <child link="${parent}_${suffix}_wheel_link" />
-    </joint>
-    <link name="${parent}_${suffix}_wheel_link">
-      <inertial>
-        <mass value="0.1" /> <!-- check jmh 20081205 -->
-        <origin xyz=" 0 0 0 " />
-        <inertia  ixx="0.012411765597" ixy="0.0" ixz="0.0"
-                  iyy="0.015218160428" iyz="0.0"
-                  izz="0.011763977943" />
-      </inertial>
-      <visual>
-        <origin xyz="0 0 0" rpy="${M_PI/2} 0 0" />
-        <geometry>
-          <cylinder radius="${wheel_radius}" length="${wheel_length}" />
-        </geometry>
-      </visual>
-      <collision>
-        <origin xyz="0 0 0" rpy="${M_PI/2} 0 0" />
-        <geometry>
-          <cylinder radius="${wheel_radius}" length="${wheel_length}" />
-        </geometry>
-      </collision>
-    </link>
-    <gazebo reference="${parent}_${suffix}_wheel_link" >
-      <elem key="mu1" value="${m}" />
-      <elem key="mu2" value="${m}" />
-      <elem key="kp"  value="100000000.0" />
-      <elem key="kd"  value="1.0" />
-    </gazebo>
-  </xacro:macro>
-  <xacro:erratic_wheel suffix="left" parent="base_link" reflect="1" offset="0" m="0.1"/>
-  <xacro:erratic_wheel suffix="left_front" parent="base_link" reflect="1" offset="0.15" m="100.1"/>
-  <xacro:erratic_wheel suffix="left_rear" parent="base_link" reflect="1" offset="-0.15" m="100.1"/>
-  <xacro:erratic_wheel suffix="right" parent="base_link" reflect="-1" offset="0" m="0.1"/>
-  <xacro:erratic_wheel suffix="right_front" parent="base_link" reflect="-1" offset="0.15" m="100.1"/>
-  <xacro:erratic_wheel suffix="right_rear" parent="base_link" reflect="-1" offset="-0.15" m="100.1"/>
-  <joint name="base_laser_joint" type="fixed">
-    <origin rpy="0 0 0" xyz="0.0 0 0.3"/>
-    <parent link="base_link"/>
-    <child link="base_laser_link"/>
-  </joint>
-  <link name="base_laser_link" type="laser">
-    <inertial>
-      <mass value="0.1"/>
-      <origin xyz="0 0 0.0"/>
-      <inertia ixx="0.1" ixy="0" ixz="0" iyy="0.1" iyz="0" izz="0.1"/>
-    </inertial>
-    <visual>
-      <origin rpy="0 0 0" xyz="0 0 0.0"/>
-      <geometry>
-        <box size="0.15 0.15 0.2"/>
-      </geometry>
-    </visual>
-    <collision>
-      <origin rpy="0 0 0" xyz="0 0 0.0"/>
-      <geometry>
-        <cylinder radius=".05" length=".05"/>
-      </geometry>
-    </collision>
-  </link>
-  <gazebo reference="base_laser_link">
-    <sensor:ray name="base_laser_link">
-      <resRange>0.01</resRange>
-      <rayCount>181</rayCount>
-      <rangeCount>181</rangeCount>
-      <laserCount>1</laserCount>
-      <origin>0.0 0.0 0.0</origin>
-      <displayRays>true</displayRays>
-      <minAngle>-90</minAngle> <!-- scans own arms if -135~+135 -->
-      <maxAngle>90</maxAngle>
-      <minRange>0.07</minRange>
-      <maxRange>10.0</maxRange>
-      <updateRate>25.0</updateRate>
-      <controller:gazebo_ros_laser name="gazebo_ros_base_laser_link_controller" plugin="libgazebo_ros_laser.so">
-        <gaussianNoise>0.005</gaussianNoise>
-        <alwaysOn>true</alwaysOn>
-        <updateRate>25.0</updateRate>
-        <topicName>base_scan</topicName>
-        <frameName>base_laser_link</frameName>
-        <interface:laser name="gazebo_ros_base_laser_link_iface"/>
-      </controller:gazebo_ros_laser>
-    </sensor:ray>
-  </gazebo>
-  <gazebo>
-    <controller:differential_position2d name="controller1">
-      <update>100</update>
-      <leftJoint>base_link_right_wheel_joint</leftJoint>
-      <rightJoint>base_link_left_wheel_joint</rightJoint>
-      <wheelSeparation>${caster_wheel_offset_y*2}</wheelSeparation>
-      <wheelDiameter>${wheel_radius*2}</wheelDiameter>
-      <torque>5</torque>
-      <interface:position name="position_iface_0"/>
-    </controller:differential_position2d>
-    <controller:gazebo_ros_p3d name="p3d_base_controller" plugin="libgazebo_ros_p3d.so">
-      <alwaysOn>true</alwaysOn>
-      <updateRate>100.0</updateRate>
-      <bodyName>base_link</bodyName>
-      <topicName>base_pose_ground_truth</topicName>
-      <gaussianNoise>0.0</gaussianNoise>
-      <frameName>map</frameName>
-      <xyzOffsets>25.7 25.7 0</xyzOffsets> <!-- initialize odometry for fake localization-->
-      <rpyOffsets>0 0 0</rpyOffsets>
-      <interface:position name="p3d_base_position"/>
-    </controller:gazebo_ros_p3d>
-  	<controller:gazebo_ros_imu name="imu_controller" plugin="libgazebo_ros_imu.so">
-      <alwaysOn>true</alwaysOn>
-      <updateRate>1000.0</updateRate>
-      <bodyName>base_link</bodyName>
-      <topicName>body_pose_ground_truth</topicName>
-      <xyzOffsets>25.65 25.65 0</xyzOffsets> <!-- option to initialize odometry for fake localization-->
-      <rpyOffsets>0 0 0</rpyOffsets>
-      <gaussianNoise>0.5</gaussianNoise>
-      <interface:position name="imu_position_iface"/>
-    </controller:gazebo_ros_imu>
-  </gazebo>
+<robot name="elektron" xmlns:sensor="http://playerstage.sourceforge.net/gazebo/xmlschema/#sensor"
+	xmlns:controller="http://playerstage.sourceforge.net/gazebo/xmlschema/#controller"
+	xmlns:xacro="http://ros.org/wiki/fixme"
+	xmlns:interface="http://playerstage.sourceforge.net/gazebo/xmlschema/#interface">
+	<property name="M_PI" value="3.14159"/>
+	<property name="base_size_x" value="0.38" />
+	<property name="base_size_y" value="0.28" />
+	<property name="base_size_z" value="0.18" />
+	<property name="wheel_radius" value="0.05" />
+	<property name="wheel_length" value="0.02" />
+	<property name="caster_wheel_offset_y" value="0.1675" />
+	<link name="base_link">
+		<inertial>
+			<mass value="15" />
+			<origin xyz="-0.0 0 ${base_size_z/2}" />
+			<inertia ixx="1.0" ixy="0.0" ixz="0.0" iyy="1.0" iyz="0.0" izz="1.0" />
+		</inertial>
+		<!--<box size="0.38 0.28 0.20" />-->
+		<visual>
+			<origin xyz="-0.0 0 0.115" rpy="0 0 0" />
+			<geometry>
+				<mesh filename="package://elektron_defs/meshes/elektron_body.blend"/>
+			</geometry>
+		</visual>
+		<collision>
+			<origin xyz="-0.0 0 0.115" rpy="0 0 0" />
+			<geometry>
+				<box size="0.30 0.28 0.20" />
+			</geometry>
+			<material name="Cyan">
+				<color rgba="0 255 255 1.0"/>
+			</material>
+		</collision>
+	</link>
+	<xacro:macro name="erratic_wheel" params="suffix parent reflect offset m">
+		<joint name="${parent}_${suffix}_wheel_joint" type="continuous">
+			<origin xyz="${offset} ${reflect*caster_wheel_offset_y} ${wheel_radius}" rpy="0	0 0"/>
+			<axis xyz="0 1 0" />
+			<anchor xyz="0 0 0" />
+			<limit effort="100" velocity="100" />
+			<joint_properties damping="0.0" friction="0.0" />
+			<parent link="${parent}" />
+			<child link="${parent}_${suffix}_wheel_link" />
+		</joint>
+		<link name="${parent}_${suffix}_wheel_link">
+			<inertial>
+				<mass value="0.1" />
+				<!-- check jmh 20081205 -->
+				<origin xyz=" 0 0 0 " />
+				<inertia ixx="0.012411765597" ixy="0.0" ixz="0.0" iyy="0.015218160428" iyz="0.0" izz="0.011763977943"/>
+			</inertial>
+			<visual>
+				<origin xyz="0 0 0" rpy="${M_PI/2} 0 0" />
+				<geometry>
+					<cylinder radius="${wheel_radius}" length="${wheel_length}" />
+				</geometry>
+			</visual>
+			<collision>
+				<origin xyz="0 0 0" rpy="${M_PI/2} 0 0" />
+				<geometry>
+					<cylinder radius="${wheel_radius}" length="${wheel_length}" />
+				</geometry>
+			</collision>
+		</link>
+		<gazebo reference="${parent}_${suffix}_wheel_link" >
+			<elem key="mu1" value="${m}" />
+			<elem key="mu2" value="${m}" />
+			<elem key="kp"  value="100000000.0" />
+			<elem key="kd"  value="1.0" />
+		</gazebo>
+	</xacro:macro>
+	<xacro:erratic_wheel suffix="left" parent="base_link" reflect="1" offset="0" m="0.1"/>
+	<xacro:erratic_wheel suffix="left_front" parent="base_link" reflect="1" offset="0.15" m="100.1"/>
+	<xacro:erratic_wheel suffix="left_rear" parent="base_link" reflect="1" offset="-0.15" m="100.1"/>
+	<xacro:erratic_wheel suffix="right" parent="base_link" reflect="-1" offset="0" m="0.1"/>
+	<xacro:erratic_wheel suffix="right_front" parent="base_link" reflect="-1" offset="0.15"
+		m="100.1"/>
+	<xacro:erratic_wheel suffix="right_rear" parent="base_link" reflect="-1" offset="-0.15"	m="100.1"/>
+	<joint name="base_laser_joint" type="fixed">
+		<origin rpy="0 0 0" xyz="0.0 0 0.3"/>
+		<parent link="base_link"/>
+		<child link="base_laser_link"/>
+	</joint>
+	<link name="base_laser_link" type="laser">
+		<inertial>
+			<mass value="0.1"/>
+			<origin xyz="0 0 0.0"/>
+			<inertia ixx="0.1" ixy="0" ixz="0" iyy="0.1" iyz="0" izz="0.1"/>
+		</inertial>
+		<visual>
+			<origin rpy="0 0 0" xyz="0 0 0.0"/>
+			<geometry>
+				<box size="0.15 0.15 0.2"/>
+			</geometry>
+		</visual>
+		<collision>
+			<origin rpy="0 0 0" xyz="0 0 0.0"/>
+			<geometry>
+				<cylinder radius=".05" length=".05"/>
+			</geometry>
+		</collision>
+	</link>
+	<gazebo reference="base_laser_link">
+		<sensor:ray name="base_laser_link">
+			<resRange>0.01</resRange>
+			<rayCount>181</rayCount>
+			<rangeCount>181</rangeCount>
+			<laserCount>1</laserCount>
+			<origin>0.0 0.0 0.0</origin>
+			<displayRays>true</displayRays>
+			<minAngle>-90</minAngle>
+			<maxAngle>90</maxAngle>
+			<minRange>0.07</minRange>
+			<maxRange>10.0</maxRange>
+			<updateRate>25.0</updateRate>
+			<controller:gazebo_ros_laser name="gazebo_ros_base_laser_link_controller"
+				plugin="libgazebo_ros_laser.so">
+				<gaussianNoise>0.005</gaussianNoise>
+				<alwaysOn>true</alwaysOn>
+				<updateRate>25.0</updateRate>
+				<topicName>base_scan</topicName>
+				<frameName>base_laser_link</frameName>
+				<interface:laser name="gazebo_ros_base_laser_link_iface"/>
+			</controller:gazebo_ros_laser>
+		</sensor:ray>
+	</gazebo>
+	<gazebo>
+		<controller:differential_position2d name="controller1">
+			<update>100</update>
+			<leftJoint>base_link_right_wheel_joint</leftJoint>
+			<rightJoint>base_link_left_wheel_joint</rightJoint>
+			<wheelSeparation>${caster_wheel_offset_y*2}</wheelSeparation>
+			<wheelDiameter>${wheel_radius*2}</wheelDiameter>
+			<torque>5</torque>
+			<interface:position name="position_iface_0"/>
+		</controller:differential_position2d>
+		<controller:gazebo_ros_p3d name="p3d_base_controller" plugin="libgazebo_ros_p3d.so">
+			<alwaysOn>true</alwaysOn>
+			<updateRate>100.0</updateRate>
+			<bodyName>base_link</bodyName>
+			<topicName>base_pose_ground_truth</topicName>
+			<gaussianNoise>0.0</gaussianNoise>
+			<frameName>map</frameName>
+			<xyzOffsets>25.7 25.7 0</xyzOffsets>
+			<!-- initialize odometry for fake localization-->
+			<rpyOffsets>0 0 0</rpyOffsets>
+			<interface:position name="p3d_base_position"/>
+		</controller:gazebo_ros_p3d>
+		<controller:gazebo_ros_imu name="imu_controller" plugin="libgazebo_ros_imu.so">
+			<alwaysOn>true</alwaysOn>
+			<updateRate>1000.0</updateRate>
+			<bodyName>base_link</bodyName>
+			<topicName>body_pose_ground_truth</topicName>
+			<xyzOffsets>25.7 25.7 0</xyzOffsets>
+			<!-- option to initialize odometry for fake localization-->
+			<rpyOffsets>0 0 0</rpyOffsets>
+			<gaussianNoise>0.5</gaussianNoise>
+			<interface:position name="imu_position_iface"/>
+		</controller:gazebo_ros_imu>
+	</gazebo>
 </robot>

Commit message: commented gyro, laser transformation updated

File: elektron_defs/robots/elektron.udrf.xacro (robot description, xacro)
@@ -79,5 +79,5 @@
 	<xacro:erratic_wheel suffix="right_rear" parent="base_link" reflect="-1" offset="-0.15"	m="100.1"/>
 	<joint name="base_laser_joint" type="fixed">
-		<origin rpy="0 0 0" xyz="0.0 0 0.3"/>
+		<origin rpy="0 0 0" xyz="0.14 0 0.3"/>
 		<parent link="base_link"/>
 		<child link="base_laser_link"/>
